Commit message: completa renderizado de 3 carritos correctamente

File: agentes_cooperacion/install/agente_pkg/share/agente_pkg/urdf/agente.xacro (robot description, xacro)
@@ -1,5 +1,5 @@
 <?xml version="1.0"?>
 <robot name="agent_robot" xmlns:xacro="http://www.ros.org/wiki/xacro">
-  <!-- parametros -->
+  <xacro:arg name="prefix" default=""/>
   <xacro:property name="wheel_radius" value="0.05"/>
   <xacro:property name="wheel_width" value="0.02"/>
@@ -8,91 +8,39 @@
   <xacro:property name="wheel_y" value="${half_base + 0.03}"/>
   <xacro:property name="wheel_x" value="${half_base}"/>
-  <!-- base del robot -->
-  <link name="base_link">
+  <link name="$(arg prefix)base_link">
     <visual>
       <origin xyz="0 0 0" rpy="0 0 0"/>
-      <geometry>
-        <box size="${base_size} ${base_size} 0.1"/>
-      </geometry>
-      <material name="blue">
-        <color rgba="1 0 0 1"/>
-      </material>
+      <geometry><box size="${base_size} ${base_size} 0.1"/></geometry>
+      <material name="blue"><color rgba="1 0 0 1"/></material>
     </visual>
   </link>
-  <!-- rueda izquierda anterior-->
-  <link name="left_wheel_a">
-    <visual>
-      <origin rpy="1.57 0 0"/>
-      <geometry>
-        <cylinder radius="${wheel_radius}" length="${wheel_width}"/>
-      </geometry>
-      <material name="black">
-        <color rgba="1 1 0 1"/>
-      </material>
-    </visual>
-  </link>
-  <!-- rueda izquierda posterior-->
-  <link name="left_wheel_p">
-    <visual>
-      <origin rpy="1.57 0 0"/>
-      <geometry>
-        <cylinder radius="${wheel_radius}" length="${wheel_width}"/>
-      </geometry>
-      <material name="black">
-        <color rgba="1 1 0 1"/>
-      </material>
-    </visual>
-  </link>
-  <!-- rueda derecha anterior-->
-  <link name="right_wheel_a">
-    <visual>
-      <origin rpy="1.57 0 0"/>
-      <geometry>
-        <cylinder radius="${wheel_radius}" length="${wheel_width}"/>
-      </geometry>
-      <material name="black">
-        <color rgba="1 1 0 1"/>
-      </material>
-    </visual>
-  </link>
-  <!-- rueda derecha posterior -->
-  <link name="right_wheel_p">
-    <visual>
-      <origin rpy="1.57 0 0"/>
-      <geometry>
-        <cylinder radius="${wheel_radius}" length="${wheel_width}"/>
-      </geometry>
-      <material name="black">
-        <color rgba="1 1 0 1"/>
-      </material>
-    </visual>
-  </link>
-  <!-- joint rueda izquierda-anterior-base -->
-  <joint name="left_wheel_joint_a" type="continuous">
-    <parent link="base_link"/>
-    <child link="left_wheel_a"/>
-    <origin xyz="${wheel_x} ${wheel_y} -${wheel_radius}"/>
-    <axis xyz="0 1 0"/>
+  <xacro:macro name="wheel" params="suffix">
+    <link name="$(arg prefix)wheel_${suffix}">
+      <visual>
+        <origin rpy="1.57 0 0"/>
+        <geometry><cylinder radius="${wheel_radius}" length="${wheel_width}"/></geometry>
+        <material name="black"><color rgba="1 1 0 1"/></material>
+      </visual>
+    </link>
+  </xacro:macro>
+  <xacro:wheel suffix="left_a"/>
+  <xacro:wheel suffix="left_p"/>
+  <xacro:wheel suffix="right_a"/>
+  <xacro:wheel suffix="right_p"/>
+  <joint name="$(arg prefix)left_wheel_joint_a" type="continuous">
+    <parent link="$(arg prefix)base_link"/><child link="$(arg prefix)wheel_left_a"/>
+    <origin xyz="${wheel_x} ${wheel_y} -${wheel_radius}"/><axis xyz="0 1 0"/>
   </joint>
-  <!-- joint rueda izquierda-posterior-base -->
-  <joint name="left_wheel_joint_p" type="continuous">
-    <parent link="base_link"/>
-    <child link="left_wheel_p"/>
-    <origin xyz="-${wheel_x} ${wheel_y} -${wheel_radius}"/>
-    <axis xyz="0 1 0"/>
+  <joint name="$(arg prefix)left_wheel_joint_p" type="continuous">
+    <parent link="$(arg prefix)base_link"/><child link="$(arg prefix)wheel_left_p"/>
+    <origin xyz="-${wheel_x} ${wheel_y} -${wheel_radius}"/><axis xyz="0 1 0"/>
   </joint>
-  <!-- joint rueda derecha-anterior-base -->
-  <joint name="right_wheel_joint_a" type="continuous">
-    <parent link="base_link"/>
-    <child link="right_wheel_a"/>
-    <origin xyz="${wheel_x} -${wheel_y} -${wheel_radius}"/>
-    <axis xyz="0 1 0"/>
+  <joint name="$(arg prefix)right_wheel_joint_a" type="continuous">
+    <parent link="$(arg prefix)base_link"/><child link="$(arg prefix)wheel_right_a"/>
+    <origin xyz="${wheel_x} -${wheel_y} -${wheel_radius}"/><axis xyz="0 1 0"/>
   </joint>
-   <!-- joint rueda derecha-posterior-base -->
-  <joint name="right_wheel_joint_p" type="continuous">
-    <parent link="base_link"/>
-    <child link="right_wheel_p"/>
-    <origin xyz="-${wheel_x} -${wheel_y} -${wheel_radius}"/>
-    <axis xyz="0 1 0"/>
+  <joint name="$(arg prefix)right_wheel_joint_p" type="continuous">
+    <parent link="$(arg prefix)base_link"/><child link="$(arg prefix)wheel_right_p"/>
+    <origin xyz="-${wheel_x} -${wheel_y} -${wheel_radius}"/><axis xyz="0 1 0"/>
   </joint>
 </robot>
